Commit message: fix(description): connect MID-360 IMU frame

File: packages/go2_description/urdf/go2_robonix.urdf (robot description, URDF)
Before this commit: robot go2_description, 44 links, 43 joints
Links:
- added link utlidar_imu
Joints:
- added joint utlidar_lidar_to_utlidar_imu: type fixed, parent utlidar_lidar, child utlidar_imu, origin xyz=0.011 0.02329 -0.04412 rpy=0 0 0

Commit message: feat(stack): publish validated Go2 voice navigation
Publish the already validated Client-to-semantic-to-Nav2-to-Go2 stack, guarded chassis ownership and stop path, generation-scoped Mapping integration, operator surfaces, and reproducible Mapping and Navigation pins.

Assisted-by: Codex:gpt-5.6-sol [TOOL Codex]

File: packages/go2_description/urdf/go2_robonix.urdf (robot description, URDF)
Before this commit: robot go2_description, 45 links, 44 joints
Joints:
- joint radar_to_utlidar_lidar: origin xyz=0 0 0 rpy=0 0 0 -> xyz=-0.005152655 0 -0.047108077 rpy=-0.001508482 -0.000981520 -2.146758680
- joint utlidar_lidar_to_utlidar_imu: origin xyz=0.011 0.02329 -0.04412 rpy=0 0 0 -> xyz=-0.007698 -0.014655 0.00667 rpy=0 0 0
